Commit message: Robot model 3dof updated for SCARA Type robot.

File: urdf/my_3dof_arm.urdf.xacro (robot description, xacro)
@@ -1,68 +1,61 @@
 <?xml version="1.0"?>
-<robot xmlns:xacro="http://ros.org/wiki/xacro" name="my_3dof_arm">
+<robot xmlns:xacro="http://ros.org/wiki/xacro" name="scara_robot">
+<!-- ROBOT v2: SCARA Type 3dof -->
   <!-- Base -->
   <link name="base_link">
     <visual>
-      <geometry><cylinder length="0.1" radius="0.05"/></geometry>
+      <geometry><cylinder length="0.25" radius="0.075"/></geometry>
       <material name="grey"><color rgba="0.7 0.7 0.7 1"/></material>
     </visual>
   </link>
-  <!-- Shoulder joint -->
+  <!-- Joint1: Base rotation -->
   <joint name="joint1" type="revolute">
     <parent link="base_link"/>
     <child link="link1"/>
-    <origin xyz="0 0 0.05" rpy="0 0 0"/>
-    <axis xyz="0 0 1"/>
-    <limit lower="-1.57" upper="1.57" effort="10" velocity="1"/>
+    <origin xyz="0 0 0.15" rpy="0 0 0"/>
+    <axis xyz="0 0 2"/>
+    <limit lower="-3.14" upper="3.14" effort="10" velocity="1"/>
   </joint>
   <link name="link1">
     <visual>
-      <geometry><box size="0.3 0.05 0.05"/></geometry>
+      <geometry><box size="0.3 0.075 0.035"/></geometry>
       <origin xyz="0.15 0 0" rpy="0 0 0"/>
       <material name="blue"><color rgba="0.2 0.6 0.9 1"/></material>
     </visual>
   </link>
-  <!-- Elbow joint -->
+  <!-- Joint2: Shoulder rotation -->
   <joint name="joint2" type="revolute">
     <parent link="link1"/>
     <child link="link2"/>
-    <origin xyz="0.3 0 0" rpy="0 0 0"/>
+    <origin xyz="0.25 0 0.030" rpy="0 0 0"/>
     <axis xyz="0 0 1"/>
-    <limit lower="-1.57" upper="1.57" effort="10" velocity="1"/>
+    <limit lower="-2.36" upper="2.36" effort="10" velocity="1"/>
   </joint>
   <link name="link2">
     <visual>
-      <geometry><box size="0.25 0.04 0.04"/></geometry>
+      <geometry><box size="0.25 0.055 0.035"/></geometry>
       <origin xyz="0.125 0 0" rpy="0 0 0"/>
       <material name="red"><color rgba="0.9 0.3 0.3 1"/></material>
     </visual>
   </link>
-  <!-- Wrist joint -->
-  <joint name="joint3" type="revolute">
+  <!-- Joint3: Z-axis -->
+  <joint name="joint3" type="prismatic">
     <parent link="link2"/>
     <child link="link3"/>
-    <origin xyz="0.25 0 0" rpy="0 0 0"/>
+    <origin xyz="0.125 0 0.015" rpy="0 0 0"/>
     <axis xyz="0 0 1"/>
-    <limit lower="-1.57" upper="1.57" effort="10" velocity="1"/>
+    <limit lower="-0.12" upper="0.08" effort="10" velocity="1"/>
   </joint>
   <link name="link3">
     <visual>
-      <geometry><box size="0.2 0.03 0.03"/></geometry>
+      <geometry><box size="0.02 0.03 0.25"/></geometry>
       <origin xyz="0.1 0 0" rpy="0 0 0"/>
-      <material name="green"><color rgba="0.3 0.9 0.3 1"/></material>
+      <material name="green"><color rgba="0.2 0.75 0.3 1"/></material>
+    </visual>
+    <visual>
+      <origin xyz="0.1 0 -0.12" rpy="0 0 0"/>
+      <geometry><sphere radius="0.020"/></geometry>
+      <material name="yellow"><color rgba="0.35 0.35 0.75 1"/></material>
     </visual>
   </link>
-  <!-- End effector -->
-  <link name="ee_link">
-    <visual>
-      <geometry><sphere radius="0.03"/></geometry>
-      <origin xyz="0.02 0 0" rpy="0 0 0"/>
-      <material name="yellow"><color rgba="0.9 0.9 0.2 1"/></material>
-    </visual>
-  </link>
-  <joint name="ee_joint" type="fixed">
-    <parent link="link3"/>
-    <child link="ee_link"/>
-    <origin xyz="0.2 0 0" rpy="0 0 0"/>
-  </joint>
 </robot>
