Commit message: URDF model height issue fix, on platform now, links intact.

File: urdf/my_3dof_arm.urdf.xacro (robot description, xacro)
@@ -5,4 +5,5 @@
   <link name="base_link">
     <visual>
+      <origin xyz="0 0 0.125" rpy="0 0 0"/>
       <geometry><cylinder length="0.25" radius="0.075"/></geometry>
       <material name="grey"><color rgba="0.7 0.7 0.7 1"/></material>
@@ -13,5 +14,5 @@
     <parent link="base_link"/>
     <child link="link1"/>
-    <origin xyz="0 0 0.15" rpy="0 0 0"/>
+    <origin xyz="0 0 0.275" rpy="0 0 0"/>
     <axis xyz="0 0 2"/>
     <limit lower="-3.14" upper="3.14" effort="10" velocity="1"/>
